Commit message: Nav2 Working

File: description/camera.xacro (robot description, xacro)
@@ -11,6 +11,5 @@
                 <box size="0.01 0.03 0.03"/>
             </geometry>
-            <material name="red">
-                <color rgba="1 0 0 1"/> </material>
+            <material name="red"/>
         </visual>
     </link>

File: description/depth_camera.xacro (robot description, xacro)
@@ -11,6 +11,5 @@
                 <box size="0.01 0.03 0.03"/>
             </geometry>
-            <material name="red">
-                <color rgba="1 0 0 1"/> </material>
+            <material name="red"/>
         </visual>
     </link>
@@ -22,5 +21,4 @@
     <link name="camera_optical_link"></link>
 <gazebo reference="camera_link">
-        <material>Gazebo/Red</material>
         <sensor name="camera" type="depth">
             <pose> 0 0 0 0 0 0 </pose>

File: description/lidar.xacro (robot description, xacro)
@@ -11,6 +11,5 @@
                 <cylinder radius="0.05" length="0.04"/>
             </geometry>
-            <material name="red">
-                <color rgba="1 0 0 1"/> </material>
+            <material name="red"/>
         </visual>
         <collision>
@@ -23,12 +22,5 @@
         </xacro:inertial_cylinder>
     </link>
-    <gazebo>
-        <plugin
-            filename="gz-sim-sensors-system" name="gz::sim::systems::Sensors">
-            <render_engine>ogre2</render_engine>
-        </plugin>
-    </gazebo>
     <gazebo reference="laser_frame">
-        <material>Gazebo/Red</material>
         <sensor name="laser" type="gpu_lidar">
             <pose> 0 0 0 0 0 0 </pose>

File: description/robot_core.xacro (robot description, xacro)
@@ -14,4 +14,7 @@
         <color rgba="0 0 0 1"/>
     </material>
+    <material name="red">
+        <color rgba="1 0 0 1"/>
+    </material>
 <!-- Base Link -->
     <link name="base_link">
@@ -22,4 +25,12 @@
         <origin xyz="-0.1 0 0"/>
     </joint>
+<!--base_footprint_link-->
+    <joint name="base_footprint_joint" type="fixed">
+        <parent link="base_link"/>
+        <child link="base_footprint"/>
+        <origin xyz = "0 0 0" rpy="0 0 0"/>
+    </joint>
+    <link name="base_footprint">
+    </link>
 <!-- Chassis Link-->
     <link name="chassis">
@@ -41,7 +52,4 @@
         </xacro:inertial_box>
     </link>
-    <gazebo reference="chassis">
-        <material>Gazebo/White</material>
-    </gazebo>
 <!--Left Wheel Joint-->
     <joint name="left_wheel_joint" type="continuous">
@@ -67,7 +75,4 @@
         </xacro:inertial_cylinder>
     </link>
-    <gazebo reference="left_wheel">
-        <material>Gazebo/Blue</material>
-    </gazebo>
 <!--Right Wheel-->
     <joint name="right_wheel_joint" type="continuous">
@@ -93,7 +98,4 @@
         </xacro:inertial_cylinder>
     </link>
-    <gazebo reference="right_wheel">
-        <material>Gazebo/Blue</material>
-    </gazebo>
     <joint name="caster_wheel_joint" type="fixed">
         <parent link="chassis"/>

Commit message: successfully added rtab & ran nav2

File: description/camera.xacro (robot description, xacro)
@@ -13,4 +13,8 @@
             <material name="red"/>
         </visual>
+        <inertial>
+            <mass value="0.01"/>
+            <inertia ixx="0.00001" ixy="0" ixz="0" iyy="0.00001" iyz="0" izz="0.00001"/>
+        </inertial>
     </link>
     <joint name="camera_optical_joint" type="fixed">
@@ -32,6 +36,6 @@
                 <image>
                     <format>R8G8B8</format>
-                    <width>640</width>
-                    <height>480</height>
+                    <width>1280</width>
+                    <height>720</height>
                 </image>
                 <clip>

File: description/depth_camera.xacro (robot description, xacro)
@@ -1,30 +1,34 @@
 <?xml version="1.0"?>
 <robot xmlns:xacro="http://www.ros.org/wiki/xacro" >
-    <joint name="camera_joint" type="fixed">
+    <joint name="depth_joint" type="fixed">
         <parent link="chassis"/>
-        <child link ="camera_link"/>
-        <origin xyz="0.305 0 0.08" rpy="0 0 0"/>
+        <child link ="depth_link"/>
+        <origin xyz="0.305 0 0.125" rpy="0 0 0"/>
     </joint>
-    <link name="camera_link">
+    <link name="depth_link">
         <visual>
             <geometry>
                 <box size="0.01 0.03 0.03"/>
             </geometry>
-            <material name="red"/>
+            <material name="purple"/>
         </visual>
+        <inertial>
+            <mass value="0.01"/>
+            <inertia ixx="0.00001" ixy="0" ixz="0" iyy="0.00001" iyz="0" izz="0.00001"/>
+        </inertial>
     </link>
-    <joint name="camera_optical_joint" type="fixed">
-        <parent link="camera_link"/>
-        <child link ="camera_optical_link"/>
+    <joint name="depth_optical_joint" type="fixed">
+        <parent link="depth_link"/>
+        <child link ="depth_optical_link"/>
         <origin xyz="0 0 0" rpy="${-pi/2} 0 ${-pi/2}"/>
     </joint>
-    <link name="camera_optical_link"></link>
-<gazebo reference="camera_link">
-        <sensor name="camera" type="depth">
+    <link name="depth_optical_link"></link>
+<gazebo reference="depth_link">
+        <sensor name="dcamera" type="depth">
             <pose> 0 0 0 0 0 0 </pose>
             <visualize>true</visualize>
             <update_rate>10</update_rate>
-            <topic>camera/image_raw</topic>
-            <gz_frame_id>camera_optical_link</gz_frame_id>
+            <topic>camera/depth/image_raw</topic>
+            <gz_frame_id>depth_optical_link</gz_frame_id>
             <min_depth>0.1</min_depth>
             <max_depth>100.0</max_depth>
@@ -33,6 +37,6 @@
                 <image>
                     <format>R8G8B8</format>
-                    <width>640</width>
-                    <height>480</height>
+                    <width>1280</width>
+                    <height>720</height>
                 </image>
                 <clip>

File: description/robot.urdf.xacro (robot description, xacro)
@@ -3,5 +3,5 @@
     <xacro:include filename="robot_core.xacro" />
     <xacro:include filename="gazebo_control.xacro" />
-    <!-- <xacro:include filename="camera.xacro" /> -->
+    <xacro:include filename="camera.xacro" />
     <xacro:include filename="depth_camera.xacro" />
     <xacro:include filename="lidar.xacro" />

File: description/robot_core.xacro (robot description, xacro)
@@ -16,4 +16,7 @@
     <material name="red">
         <color rgba="1 0 0 1"/>
+    </material>
+    <material name="purple" >
+        <color rgba="0.49411764705882355 0.11764705882352941 0.611764705882353 1.0" />
     </material>
 <!-- Base Link -->
